Commit message: Add RGB-D camera to my_robot

File: my_robot/urdf/my_robot.xacro (robot description, xacro)
@@ -120,9 +120,9 @@
   <joint type="fixed" name="camera_joint">
     <origin xyz="0.2 0 0" rpy="0 0 0"/>
-    <child link="camera"/>
-    <parent link="chassis"/>
-    <axis xyz="0 1 0" rpy="0 0 0"/>
-  </joint>
-  <link name='camera'>
+    <child link="camera_link"/>
+    <parent link="chassis"/>
+    <axis xyz="0 1 0" rpy="0 0 0"/>
+  </joint>
+  <link name='camera_link'>
     <inertial>
       <mass value="0.1"/>
@@ -176,4 +176,32 @@
     </visual>
   </link>
+  <link name="camera_link_optical">
+    <!-- <inertial> -->
+    <!--   <mass value="1e-5"/> -->
+    <!--   <origin xyz="0.05 0.05 0.05" rpy="0 0 0"/> -->
+    <!--   <inertia -->
+    <!--       ixx="1e-6" ixy="0" ixz="0" -->
+    <!--       iyy="1e-6" iyz="0" -->
+    <!--       izz="1e-6" -->
+    <!--   /> -->
+    <!-- </inertial> -->
+    <!-- <collision name='hokuyo_collision'> -->
+    <!--   <origin xyz="0 0 0" rpy="0 0 0"/> -->
+    <!--   <geometry> -->
+    <!--     <box size="0.1 0.1 0.1"/> -->
+    <!--   </geometry> -->
+    <!-- </collision> -->
+    <!-- <visual name='hokuyo_visual'> -->
+    <!--   <origin xyz="0 0 0" rpy="0 0 0"/> -->
+    <!--   <geometry> -->
+    <!--     <mesh filename='package://my_robot/meshes/hokuyo.dae'/> -->
+    <!--   </geometry> -->
+    <!-- </visual> -->
+  </link>
+  <joint name="camera_optical_joint" type="fixed">
+    <origin xyz="0 0 0" rpy="-1.5707 0 -1.5707"/>
+    <child link="camera_link_optical"/>
+    <parent link="camera_link"/>
+  </joint>
   <gazebo reference="left_wheel">
     <material>Gazebo/DarkGrey</material>
